Commit message: /LaserScan is online
Rviz now displays LiDAR data. frame still moves with the robot though.

File: robot/x_drive.urdf.xacro (robot description, xacro)
@@ -39,5 +39,5 @@
 	<!--Sensor links-->
 	<link name="imu_link"/>
-	<link name="base_scan">
+	<link name="laser_frame">
 			<visual>
 				<origin xyz="0 0 0.0" rpy="0 0 0"/>
@@ -149,7 +149,37 @@
 	<joint name="scan_joint" type='fixed'>
 		<parent link="base_link"/>
-		<child link="base_scan"/>
+		<child link="laser_frame"/>
 		<origin xyz="0 0 0.1" rpy="0 0 0"/>
 	</joint>
+	<!-- Sensor Gazebo Tag-->
+    <gazebo reference="laser_frame">
+        <sensor name="laser" type="gpu_lidar">
+            <pose>0 0 0 0 0 0</pose>
+            <always_on>true</always_on>
+            <visualize>true</visualize>
+            <update_rate>10</update_rate>
+            <topic>LaserScan</topic>
+            <lidar>
+                <scan>
+                    <horizontal>
+						<samples>720</samples>
+						<resolution>1</resolution>
+						<min_angle>-3.14</min_angle>
+						<max_angle>3.14</max_angle>
+                    </horizontal>
+                </scan>
+                <range>
+                    <min>0.05</min>
+                    <max>10.0</max>
+                    <resolution>0.01</resolution>
+                </range>
+                <noise>
+                    <type>gaussian</type>
+                    <mean>0.0</mean>
+                    <stddev>0.01</stddev>
+                </noise>
+            </lidar>
+        </sensor>
+    </gazebo>
 	<!-- ROS 2 Control-->
 	<ros2_control name="GazeboSystem" type="system">
@@ -178,5 +208,5 @@
  		</joint>
 	</ros2_control>
-	<!-- gazebo stuff -->
+	<!-- Gazebo Sim Plugins -->
 	<gazebo>
   		<plugin filename="gz_ros2_control-system" name="gz_ros2_control::GazeboSimROS2ControlPlugin">

Commit message: fixed urdf issue

File: robot/x_drive.urdf.xacro (robot description, xacro)
@@ -1,88 +1,88 @@
 <?xml version='1.0'?>
 <robot name="x_drive" xmlns:xacro="http://www.ros.org/wiki/xacro" xmlns:gz="http://gazebosim.org/schema">
-	<static>false</static>
-	<!-- properties-->
-	<xacro:property name="model_path" value="package://robot_description/models"/>
-	<xacro:property name="package_path" value="package://robot_gazebo/config"/>
-	<xacro:property name="wheel_offs" value="0.14"/>
-	<xacro:property name="wheel_rad" value="0.01375"/>
-	<xacro:property name="wheel_width" value="0.02159"/>
-	<!--world link-->
-	<link name='base_footprint'/>
-	<!--chassis link-->
-	<link name="base_link">
-		<visual>
-			<geometry>
-				<mesh filename='${model_path}/chassis.dae'/>
-			</geometry>
-			<material name="pink">
+    <static>false</static>
+    <!-- properties-->
+    <xacro:property name="model_path" value="package://robot_description/models"/>
+    <xacro:property name="package_path" value="package://robot_gazebo/config"/>
+    <xacro:property name="wheel_offs" value="0.14"/>
+    <xacro:property name="wheel_rad" value="0.01375"/>
+    <xacro:property name="wheel_width" value="0.02159"/>
+    <!--world link-->
+    <link name='base_footprint'/>
+    <!--chassis link-->
+    <link name="base_link">
+        <visual>
+            <geometry>
+                <mesh filename='${model_path}/chassis.dae'/>
+            </geometry>
+            <material name="pink">
                 <color rgba="0.93 0.28 0.60 1.0"/>
-			</material>
-		</visual>
-		<collision>
-			<geometry>
-				<mesh filename='${model_path}/chassis.dae'/>
-			</geometry>
-		</collision>
-		<inertial>
+            </material>
+        </visual>
+        <collision>
+            <geometry>
+                <mesh filename='${model_path}/chassis.dae'/>
+            </geometry>
+        </collision>
+        <inertial>
             <origin xyz="0 0 0" rpy="0 0 0"/>
             <mass value="4.54"/>
            <inertia
-      			ixx="0.05487"
-				ixy="0.0"
-				ixz="0.0"
-				iyy="0.05487"
-				iyz="0.0"
-				izz="0.10974"/>
-    		</inertial>
-	</link>
-	<!--Sensor links-->
-	<link name="imu_link"/>
-	<link name="laser_frame">
-			<visual>
-				<origin xyz="0 0 0.0" rpy="0 0 0"/>
-				<geometry>
-					<cylinder length="0.0315" radius="0.055"/>
-				</geometry>
-				<material name="dark_grey">
-					<color rgba="0.2 0.2 0.2 1.0"/>
-				</material>
-			</visual>
-			<collision>
-				<origin xyz="0.015 0 -0.0065" rpy="0 0 0"/>
-				<geometry>
-					<cylinder length="0.0315" radius="0.055"/>
-				</geometry>
-			</collision>
-			<inertial>
-				<origin xyz="0 0 0" />
-				<mass value="0.114" />
-				<inertia
-				ixx="0.001"
-				ixy="0.0"
-				ixz="0.0"
-				iyy="0.001"
-				iyz="0.0"
-				izz="0.001"/>
-			</inertial>
-	</link>
-	<!-- wheels -->
-	<xacro:macro name="wheel_link" params="name">
-		<link name="${name}">
-			<visual>
-			<origin xyz="0 0 0" rpy="${pi/2} 0 0"/>
-				<geometry>
-					<cylinder radius='${wheel_rad*2}' length='${wheel_width}' />
-				</geometry>
-				<material name="dark_grey">
-					<color rgba="0.2 0.2 0.2 1.0"/>
-				</material>
-			</visual>
-			<collision>
-			<origin xyz="0 0 0" rpy="${pi/2} 0 0"/>
-				<geometry>
-					<cylinder radius='${wheel_rad*2}' length='${wheel_width}' />
-				</geometry>
-					<surface>
+                  ixx="0.05487"
+                ixy="0.0"
+                ixz="0.0"
+                iyy="0.05487"
+                iyz="0.0"
+                izz="0.10974"/>
+            </inertial>
+    </link>
+    <!--Sensor links-->
+    <link name="imu_link"/>
+    <link name="laser_frame">
+            <visual>
+                <origin xyz="0 0 0.0" rpy="0 0 0"/>
+                <geometry>
+                    <cylinder length="0.0315" radius="0.055"/>
+                </geometry>
+                <material name="dark_grey">
+                    <color rgba="0.2 0.2 0.2 1.0"/>
+                </material>
+            </visual>
+            <collision>
+                <origin xyz="0.015 0 -0.0065" rpy="0 0 0"/>
+                <geometry>
+                    <cylinder length="0.0315" radius="0.055"/>
+                </geometry>
+            </collision>
+            <inertial>
+                <origin xyz="0 0 0" />
+                <mass value="0.114" />
+                <inertia
+                ixx="0.001"
+                ixy="0.0"
+                ixz="0.0"
+                iyy="0.001"
+                iyz="0.0"
+                izz="0.001"/>
+            </inertial>
+    </link>
+    <!-- wheels -->
+    <xacro:macro name="wheel_link" params="name">
+        <link name="${name}">
+            <visual>
+            <origin xyz="0 0 0" rpy="${pi/2} 0 0"/>
+                <geometry>
+                    <cylinder radius='${wheel_rad*2}' length='${wheel_width}' />
+                </geometry>
+                <material name="dark_grey">
+                    <color rgba="0.2 0.2 0.2 1.0"/>
+                </material>
+            </visual>
+            <collision>
+            <origin xyz="0 0 0" rpy="${pi/2} 0 0"/>
+                <geometry>
+                    <cylinder radius='${wheel_rad*2}' length='${wheel_width}' />
+                </geometry>
+                    <surface>
                     <friction>
                         <ode>
@@ -93,124 +93,124 @@
                     </friction>
                 </surface>
-			</collision>
-			<inertial>
-            	<origin xyz="0 0 0" rpy="0 0 0"/>
-            	<mass value="0.070"/>
-				<inertia
-      			ixx="0.001"
-				ixy="0.0"
-				ixz="0.0"
-				iyy="0.001"
-				iyz="0.0"
-				izz="0.001"/>
-        	</inertial>
-		</link>
-	</xacro:macro>
-	<xacro:wheel_link name="wheel_a"/>
-	<xacro:wheel_link name="wheel_b"/>
-	<xacro:wheel_link name="wheel_c"/>
-	<xacro:wheel_link name="wheel_d"/>
-	<!--Sensor links-->
-	<link name="imu_link"/>
-	<link name="base_scan">
-			<visual>
-				<origin xyz="0 0 0.0" rpy="0 0 0"/>
-				<geometry>
-					<cylinder length="0.0315" radius="0.055"/>
-				</geometry>
-				<material name="dark_grey">
-					<color rgba="0.2 0.2 0.2 1.0"/>
-				</material>
-			</visual>
-			<collision>
-				<origin xyz="0.015 0 -0.0065" rpy="0 0 0"/>
-				<geometry>
-					<cylinder length="0.0315" radius="0.055"/>
-				</geometry>
-			</collision>
-			<inertial>
-				<origin xyz="0 0 0" />
-				<mass value="0.114" />
-				<inertia
-				ixx="0.001"
-				ixy="0.0"
-				ixz="0.0"
-				iyy="0.001"
-				iyz="0.0"
-				izz="0.001"/>
-			</inertial>
-	</link>
-	<!-- joints -->
-	<joint name="world_2_chassis" type='fixed'>
-		<origin xyz="0 0 0.025" rpy="0 0 0"/>
-		<parent link='base_footprint'/>
-		<child link='base_link'/>
-	</joint>
-	<joint name="chassis_to_wheel_a" type="continuous">
+            </collision>
+            <inertial>
+                <origin xyz="0 0 0" rpy="0 0 0"/>
+                <mass value="0.070"/>
+                <inertia
+                ixx="0.001"
+                ixy="0.0"
+                ixz="0.0"
+                iyy="0.001"
+                iyz="0.0"
+                izz="0.001"/>
+            </inertial>
+        </link>
+    </xacro:macro>
+    <xacro:wheel_link name="wheel_a"/>
+    <xacro:wheel_link name="wheel_b"/>
+    <xacro:wheel_link name="wheel_c"/>
+    <xacro:wheel_link name="wheel_d"/>
+    <!-- joints -->
+    <joint name="world_2_chassis" type='fixed'>
+        <origin xyz="0 0 0.025" rpy="0 0 0"/>
+        <parent link='base_footprint'/>
+        <child link='base_link'/>
+    </joint>
+    <joint name="chassis_to_wheel_a" type="continuous">
         <origin xyz="-${wheel_offs} ${wheel_offs} ${wheel_rad}" rpy="0 0 ${pi/4}"/>
         <parent link="base_link"/>
         <child link="wheel_a"/>
-		<axis xyz="0 1 0"/>
-    </joint>
-	<joint name="chassis_to_wheel_b" type="continuous">
+        <axis xyz="0 1 0"/>
+    </joint>
+    <joint name="chassis_to_wheel_b" type="continuous">
         <origin xyz="${wheel_offs} -${wheel_offs} ${wheel_rad}" rpy="0 0 ${-3* (pi/4)}"/>
         <parent link="base_link"/>
         <child link="wheel_b"/>
-		<axis xyz="0 1 0"/>
-    </joint>
-	<joint name="chassis_to_wheel_c" type="continuous">
+        <axis xyz="0 1 0"/>
+    </joint>
+    <joint name="chassis_to_wheel_c" type="continuous">
         <origin xyz="${wheel_offs} ${wheel_offs} ${wheel_rad}" rpy="0 0 -${pi/4}"/>
         <parent link="base_link"/>
         <child link="wheel_c"/>
-		<axis xyz="0 1 0"/>
-    </joint>
-	<joint name="chassis_to_wheel_d" type="continuous">
+        <axis xyz="0 1 0"/>
+    </joint>
+    <joint name="chassis_to_wheel_d" type="continuous">
         <origin xyz="-${wheel_offs} -${wheel_offs} ${wheel_rad}" rpy="0 0 ${3 *(pi/4)}"/>
         <parent link="base_link"/>
         <child link="wheel_d"/>
-		<axis xyz="0 1 0"/>
-    </joint>
-	<!--Sensor Joints-->
-	<joint name="imu_joint" type="fixed">
-		<parent link="base_link"/>
-		<child link="imu_link"/>
-		<origin xyz="0 0 0.04" rpy="0 0 0"/>
-	</joint>
-	<joint name="scan_joint" type="fixed">
-     	<parent link="base_link"/>
-     	<child link="base_scan"/>
-    	<origin xyz="0 0 0.2" rpy="0 0 0"/>
-  	</joint>
-	<!-- ROS 2 Control-->
-	<ros2_control name="GazeboSystem" type="system">
-	    <hardware>
+        <axis xyz="0 1 0"/>
+    </joint>
+    <!--Sensor Joints-->
+    <joint name="imu_joint" type="fixed">
+        <parent link="base_link"/>
+        <child link="imu_link"/>
+        <origin xyz="0 0 0.04" rpy="0 0 0"/>
+    </joint>
+    <joint name="laser_joint" type="fixed">
+         <parent link="base_link"/>
+         <child link="laser_frame"/>
+        <origin xyz="0 0 0.2" rpy="0 0 0"/>
+      </joint>
+    <!-- ROS 2 Control-->
+    <ros2_control name="GazeboSystem" type="system">
+        <hardware>
             <plugin>gz_ros2_control/GazeboSimSystem</plugin>
         </hardware>
-		<joint name="chassis_to_wheel_a">
-   			<command_interface name="velocity"/>
-			<state_interface name="position"/>
-			<state_interface name="velocity"/>
- 		</joint>
-		<joint name="chassis_to_wheel_b">
-   			<command_interface name="velocity"/>
-			<state_interface name="position"/>
-			<state_interface name="velocity"/>
- 		</joint>
-		<joint name="chassis_to_wheel_c">
-   			<command_interface name="velocity"/>
-			<state_interface name="position"/>
-			<state_interface name="velocity"/>
- 		</joint>
-		<joint name="chassis_to_wheel_d">
-   			<command_interface name="velocity"/>
-			<state_interface name="position"/>
-			<state_interface name="velocity"/>
- 		</joint>
-	</ros2_control>
-	<!-- Gazebo Sim Plugins -->
-	<gazebo>
-  		<plugin filename="gz_ros2_control-system" name="gz_ros2_control::GazeboSimROS2ControlPlugin">
-			<parameters>$(find robot_gazebo)/config/omni_wheel_params.yaml</parameters>
-  		</plugin>
-	</gazebo>
+        <joint name="chassis_to_wheel_a">
+               <command_interface name="velocity"/>
+            <state_interface name="position"/>
+            <state_interface name="velocity"/>
+         </joint>
+        <joint name="chassis_to_wheel_b">
+               <command_interface name="velocity"/>
+            <state_interface name="position"/>
+            <state_interface name="velocity"/>
+         </joint>
+        <joint name="chassis_to_wheel_c">
+               <command_interface name="velocity"/>
+            <state_interface name="position"/>
+            <state_interface name="velocity"/>
+         </joint>
+        <joint name="chassis_to_wheel_d">
+               <command_interface name="velocity"/>
+            <state_interface name="position"/>
+            <state_interface name="velocity"/>
+         </joint>
+    </ros2_control>
+    <!-- Gazebo Sim Plugins -->
+    <gazebo>
+          <plugin filename="gz_ros2_control-system" name="gz_ros2_control::GazeboSimROS2ControlPlugin">
+            <parameters>$(find robot_gazebo)/config/omni_wheel_params.yaml</parameters>
+          </plugin>
+    </gazebo>
+    <!-- Sensor Gazebo Tag-->
+    <gazebo reference="laser_frame">
+        <sensor name="laser" type="gpu_lidar">
+            <pose>0 0 0 0 0 0</pose>
+            <always_on>true</always_on>
+            <visualize>true</visualize>
+            <update_rate>10</update_rate>
+            <topic>LaserScan</topic>
+            <lidar>
+                <scan>
+                    <horizontal>
+                        <samples>720</samples>
+                        <resolution>1</resolution>
+                        <min_angle>-3.14</min_angle>
+                        <max_angle>3.14</max_angle>
+                    </horizontal>
+                </scan>
+                <range>
+                    <min>0.05</min>
+                    <max>10.0</max>
+                    <resolution>0.01</resolution>
+                </range>
+                <noise>
+                    <type>gaussian</type>
+                    <mean>0.0</mean>
+                    <stddev>0.01</stddev>
+                </noise>
+            </lidar>
+        </sensor>
+    </gazebo>
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
Commit message: everyhting launched correctly

File: robot/x_drive.urdf.xacro (robot description, xacro)
@@ -14,5 +14,5 @@
         <visual>
             <geometry>
-                <mesh filename='${model_path}/chassis.dae'/>
+                <mesh filename='${model_path}/chassis-v2.dae'/>
             </geometry>
             <material name="pink">

Commit message: nav2 launches with no errors, robot stuck in wall

File: robot/x_drive.urdf.xacro (robot description, xacro)
@@ -9,7 +9,7 @@
     <xacro:property name="wheel_width" value="0.02159"/>
     <!--world link-->
-    <link name='base_footprint'/>
+    <link name='base_link'/>
     <!--chassis link-->
-    <link name="base_link">
+    <link name="chassis">
         <visual>
             <geometry>
@@ -114,10 +114,10 @@
     <joint name="world_2_chassis" type='fixed'>
         <origin xyz="0 0 0.025" rpy="0 0 0"/>
-        <parent link='base_footprint'/>
-        <child link='base_link'/>
+        <parent link='base_link'/>
+        <child link='chassis'/>
     </joint>
     <joint name="chassis_to_wheel_a" type="continuous">
         <origin xyz="-${wheel_offs} ${wheel_offs} ${wheel_rad}" rpy="0 0 ${pi/4}"/>
-        <parent link="base_link"/>
+        <parent link="chassis"/>
         <child link="wheel_a"/>
         <axis xyz="0 1 0"/>
@@ -125,5 +125,5 @@
     <joint name="chassis_to_wheel_b" type="continuous">
         <origin xyz="${wheel_offs} -${wheel_offs} ${wheel_rad}" rpy="0 0 ${-3* (pi/4)}"/>
-        <parent link="base_link"/>
+        <parent link="chassis"/>
         <child link="wheel_b"/>
         <axis xyz="0 1 0"/>
@@ -131,5 +131,5 @@
     <joint name="chassis_to_wheel_c" type="continuous">
         <origin xyz="${wheel_offs} ${wheel_offs} ${wheel_rad}" rpy="0 0 -${pi/4}"/>
-        <parent link="base_link"/>
+        <parent link="chassis"/>
         <child link="wheel_c"/>
         <axis xyz="0 1 0"/>
@@ -137,5 +137,5 @@
     <joint name="chassis_to_wheel_d" type="continuous">
         <origin xyz="-${wheel_offs} -${wheel_offs} ${wheel_rad}" rpy="0 0 ${3 *(pi/4)}"/>
-        <parent link="base_link"/>
+        <parent link="chassis"/>
         <child link="wheel_d"/>
         <axis xyz="0 1 0"/>
@@ -143,10 +143,10 @@
     <!--Sensor Joints-->
     <joint name="imu_joint" type="fixed">
-        <parent link="base_link"/>
+        <parent link="chassis"/>
         <child link="imu_link"/>
         <origin xyz="0 0 0.04" rpy="0 0 0"/>
     </joint>
     <joint name="laser_joint" type="fixed">
-         <parent link="base_link"/>
+         <parent link="chassis"/>
          <child link="laser_frame"/>
         <origin xyz="0 0 0.2" rpy="0 0 0"/>

Commit message: nav2 is working!

File: robot/x_drive.urdf.xacro (robot description, xacro)
@@ -9,7 +9,7 @@
     <xacro:property name="wheel_width" value="0.02159"/>
     <!--world link-->
-    <link name='base_link'/>
-    <!--chassis link-->
-    <link name="chassis">
+    <link name='base_footprint'/>
+    <!--base_link link-->
+    <link name="base_link">
         <visual>
             <geometry>
@@ -112,12 +112,12 @@
     <xacro:wheel_link name="wheel_d"/>
     <!-- joints -->
-    <joint name="world_2_chassis" type='fixed'>
+    <joint name="footprint_2_link" type='fixed'>
         <origin xyz="0 0 0.025" rpy="0 0 0"/>
-        <parent link='base_link'/>
-        <child link='chassis'/>
+        <parent link='base_footprint'/>
+        <child link='base_link'/>
     </joint>
     <joint name="chassis_to_wheel_a" type="continuous">
         <origin xyz="-${wheel_offs} ${wheel_offs} ${wheel_rad}" rpy="0 0 ${pi/4}"/>
-        <parent link="chassis"/>
+        <parent link="base_link"/>
         <child link="wheel_a"/>
         <axis xyz="0 1 0"/>
@@ -125,5 +125,5 @@
     <joint name="chassis_to_wheel_b" type="continuous">
         <origin xyz="${wheel_offs} -${wheel_offs} ${wheel_rad}" rpy="0 0 ${-3* (pi/4)}"/>
-        <parent link="chassis"/>
+        <parent link="base_link"/>
         <child link="wheel_b"/>
         <axis xyz="0 1 0"/>
@@ -131,5 +131,5 @@
     <joint name="chassis_to_wheel_c" type="continuous">
         <origin xyz="${wheel_offs} ${wheel_offs} ${wheel_rad}" rpy="0 0 -${pi/4}"/>
-        <parent link="chassis"/>
+        <parent link="base_link"/>
         <child link="wheel_c"/>
         <axis xyz="0 1 0"/>
@@ -137,5 +137,5 @@
     <joint name="chassis_to_wheel_d" type="continuous">
         <origin xyz="-${wheel_offs} -${wheel_offs} ${wheel_rad}" rpy="0 0 ${3 *(pi/4)}"/>
-        <parent link="chassis"/>
+        <parent link="base_link"/>
         <child link="wheel_d"/>
         <axis xyz="0 1 0"/>
@@ -143,10 +143,10 @@
     <!--Sensor Joints-->
     <joint name="imu_joint" type="fixed">
-        <parent link="chassis"/>
+        <parent link="base_link"/>
         <child link="imu_link"/>
         <origin xyz="0 0 0.04" rpy="0 0 0"/>
     </joint>
     <joint name="laser_joint" type="fixed">
-         <parent link="chassis"/>
+         <parent link="base_link"/>
          <child link="laser_frame"/>
         <origin xyz="0 0 0.2" rpy="0 0 0"/>
@@ -186,10 +186,11 @@
     <!-- Sensor Gazebo Tag-->
     <gazebo reference="laser_frame">
-        <sensor name="laser" type="gpu_lidar">
+        <sensor name="lidar" type="gpu_lidar">
             <pose>0 0 0 0 0 0</pose>
             <always_on>true</always_on>
             <visualize>true</visualize>
             <update_rate>10</update_rate>
-            <topic>LaserScan</topic>
+            <topic>scan</topic>
+            <gz_frame_id>laser_frame</gz_frame_id>
             <lidar>
                 <scan>

Commit message: linear driving looks better

File: robot/x_drive.urdf.xacro (robot description, xacro)
@@ -6,5 +6,5 @@
     <xacro:property name="package_path" value="package://robot_gazebo/config"/>
     <xacro:property name="wheel_offs" value="0.14"/>
-    <xacro:property name="wheel_rad" value="0.01375"/>
+    <xacro:property name="wheel_rad" value="0.03493"/>
     <xacro:property name="wheel_width" value="0.02159"/>
     <!--world link-->
@@ -13,6 +13,12 @@
     <link name="base_link">
         <visual>
+            <!--
             <geometry>
                 <mesh filename='${model_path}/chassis-v2.dae'/>
+            </geometry>
+-->
+            <origin xyz="0 0 0.25" rpy="0 0 0"/>
+            <geometry>
+                <cylinder length="0.0315" radius="0.055"/>
             </geometry>
             <material name="pink">
@@ -21,6 +27,12 @@
         </visual>
         <collision>
+        <!--
             <geometry>
                 <mesh filename='${model_path}/chassis.dae'/>
+            </geometry>
+        -->
+            <origin xyz="0 0 0.25" rpy="0 0 0"/>
+            <geometry>
+                <cylinder length="0.0315" radius="0.055"/>
             </geometry>
         </collision>
@@ -73,5 +85,5 @@
             <origin xyz="0 0 0" rpy="${pi/2} 0 0"/>
                 <geometry>
-                    <cylinder radius='${wheel_rad*2}' length='${wheel_width}' />
+                    <cylinder radius='${wheel_rad}' length='${wheel_width}' />
                 </geometry>
                 <material name="dark_grey">
@@ -82,5 +94,5 @@
             <origin xyz="0 0 0" rpy="${pi/2} 0 0"/>
                 <geometry>
-                    <cylinder radius='${wheel_rad*2}' length='${wheel_width}' />
+                    <cylinder radius='${wheel_rad}' length='${wheel_width}' />
                 </geometry>
                     <surface>
