Commit message: WIP on 15-fix-driving-behavior

File: robot/x_drive.urdf.xacro (robot description, xacro)
@@ -6,5 +6,5 @@
     <xacro:property name="package_path" value="package://robot_gazebo/config"/>
     <xacro:property name="wheel_offs" value="0.14"/>
-    <xacro:property name="wheel_rad" value="0.03493"/>
+    <xacro:property name="wheel_rad" value="0.0349253"/>
     <xacro:property name="wheel_width" value="0.02159"/>
     <!--world link-->
@@ -96,13 +96,4 @@
                     <cylinder radius='${wheel_rad}' length='${wheel_width}' />
                 </geometry>
-                    <surface>
-                    <friction>
-                        <ode>
-                            <mu>1.0</mu>
-                            <mu2>0.01</mu2>
-                            <fdir1>1 0 0</fdir1>
-                        </ode>
-                    </friction>
-                </surface>
             </collision>
             <inertial>
@@ -118,4 +109,12 @@
             </inertial>
         </link>
+		<gazebo reference="${name}">
+			<mu1 value="0.2"/>
+			<mu2 value="1.5"/>
+			<kp value="10000000.0" />
+			<kd value="10000.0" />
+			<fdir1 value="0 0 1"/>
+			<maxContacts value= "1"/>
+		</gazebo>
     </xacro:macro>
     <xacro:wheel_link name="wheel_a"/>

Commit message: not my commit...

File: robot/x_drive.urdf.xacro (robot description, xacro)
@@ -6,5 +6,5 @@
     <xacro:property name="package_path" value="package://robot_gazebo/config"/>
     <xacro:property name="wheel_offs" value="0.14"/>
-    <xacro:property name="wheel_rad" value="0.03493"/>
+     <xacro:property name="wheel_rad" value="0.0349253"/>
     <xacro:property name="wheel_width" value="0.02159"/>
     <!--world link-->
@@ -17,5 +17,5 @@
                 <mesh filename='${model_path}/chassis-v2.dae'/>
             </geometry>
--->
+            -->
             <origin xyz="0 0 0.25" rpy="0 0 0"/>
             <geometry>
@@ -27,9 +27,9 @@
         </visual>
         <collision>
-        <!--
+            <!--
             <geometry>
                 <mesh filename='${model_path}/chassis.dae'/>
             </geometry>
-        -->
+            -->
             <origin xyz="0 0 0.25" rpy="0 0 0"/>
             <geometry>
@@ -96,13 +96,4 @@
                     <cylinder radius='${wheel_rad}' length='${wheel_width}' />
                 </geometry>
-                    <surface>
-                    <friction>
-                        <ode>
-                            <mu>1.0</mu>
-                            <mu2>0.01</mu2>
-                            <fdir1>1 0 0</fdir1>
-                        </ode>
-                    </friction>
-                </surface>
             </collision>
             <inertial>
@@ -118,4 +109,12 @@
             </inertial>
         </link>
+    <gazebo reference="${name}">
+        <mu1 value="0.2"/>
+        <mu2 value="1.5"/>
+        <kp value="10000000.0" />
+        <kd value="10000.0" />
+        <fdir1 value="0 0 1"/>
+        <maxContacts value= "1"/>
+    </gazebo>
     </xacro:macro>
     <xacro:wheel_link name="wheel_a"/>

Commit message: multicam working, 50% RTK

File: robot/x_drive.urdf.xacro (robot description, xacro)
@@ -6,5 +6,5 @@
     <xacro:property name="package_path" value="package://robot_gazebo/config"/>
     <xacro:property name="wheel_offs" value="0.14"/>
-     <xacro:property name="wheel_rad" value="0.0349253"/>
+    <xacro:property name="wheel_rad" value="0.0349253"/>
     <xacro:property name="wheel_width" value="0.02159"/>
     <!--world link-->
@@ -18,7 +18,7 @@
             </geometry>
             -->
-            <origin xyz="0 0 0.25" rpy="0 0 0"/>
-            <geometry>
-                <cylinder length="0.0315" radius="0.055"/>
+            <origin xyz="0 0 0.05" rpy="0 0 0"/>
+            <geometry>
+                <box size='0.20 0.20 0.02'/>
             </geometry>
             <material name="pink">
@@ -122,5 +122,75 @@
     <xacro:wheel_link name="wheel_c"/>
     <xacro:wheel_link name="wheel_d"/>
-    <!-- joints -->
+    <!-- Camera Xacro -->
+    <xacro:macro name='usb_cam' params='camera_name xyz rpy px_w px_h'>
+        <link name='${camera_name}_link'>
+            <visual>
+                <geometry>
+                    <box size='0.02 0.02 0.02'/>
+                </geometry>
+                <material name="dark_grey">
+                    <color rgba="0.2 0.2 0.2 1.0"/>
+                </material>
+            </visual>
+            <collision>
+                <geometry>
+                    <box size='0.02 0.02 0.02'/>
+                </geometry>
+                <material name="dark_grey">
+                    <color rgba="0.2 0.2 0.2 1.0"/>
+                </material>
+            </collision>
+            <inertial>
+                <origin xyz="0 0 0" rpy="0 0 0"/>
+                <mass value="0.01"/>
+                <inertia
+                    ixx="0.000001"
+                    ixy="0.0"
+                    ixz="0.0"
+                    iyy="0.000001"
+                    iyz="0.0"
+                    izz="0.000001"/>
+            </inertial>
+        </link>
+        <joint name="${camera_name}_joint" type="fixed">
+            <parent link="base_link"/>
+            <child link="${camera_name}_link"/>
+            <origin xyz="${xyz}" rpy="${rpy}"/>
+        </joint>
+        <link name="${camera_name}_link_optical"/>
+        <joint name="${camera_name}_optical_joint" type="fixed">
+            <parent link="${camera_name}_link"/>
+            <child link="${camera_name}_link_optical"/>
+            <origin xyz="0 0 0" rpy="-1.5708 0 -1.5708"/>
+        </joint>
+        <gazebo reference='${camera_name}_link'>
+            <sensor name='${camera_name}_sensor' type="camera">
+                <pose>0 0 0 0 0 0</pose>
+                <camera>
+                    <horizontal_fov>1.047</horizontal_fov>
+                    <image>
+                        <width>${px_w}</width>
+                        <height>${px_h}</height>
+                        <format>R8G8B8</format>
+                    </image>
+                    <clip>
+                        <near>0.1</near>
+                        <far>100</far>
+                    </clip>
+                </camera>
+                <always_on>true</always_on>
+                <update_rate>30</update_rate>
+                <visualize>true</visualize>
+                <topic>/${camera_name}/image_raw</topic>
+                <gz_frame_id>${camera_name}_link_optical</gz_frame_id>
+            </sensor>
+        </gazebo>
+    </xacro:macro>
+    <xacro:usb_cam camera_name='cam1' px_w='1920' px_h='1200' xyz='0.1 0 0.1' rpy='0 0 0'/>
+    <xacro:usb_cam camera_name='cam2' px_w='1920' px_h='1200' xyz='-0.1 0 0.1' rpy='0 0 ${pi}'/>
+    <xacro:usb_cam camera_name='cam3' px_w='1920' px_h='1200' xyz='0 0.1 0.1' rpy='0 0 ${pi/2}'/>
+    <xacro:usb_cam camera_name='cam4' px_w='1920' px_h='1200' xyz='0 -0.1 0.1' rpy='0 0 -${pi/2}'/>
+    <!-- make sure to update ROS bridge in spawn_robot.launch.py! -->
+    <!-- Joints -->
     <joint name="footprint_2_link" type='fixed'>
         <origin xyz="0 0 0.025" rpy="0 0 0"/>
@@ -159,8 +229,8 @@
     </joint>
     <joint name="laser_joint" type="fixed">
-         <parent link="base_link"/>
-         <child link="laser_frame"/>
+        <parent link="base_link"/>
+        <child link="laser_frame"/>
         <origin xyz="0 0 0.2" rpy="0 0 0"/>
-      </joint>
+    </joint>
     <!-- ROS 2 Control-->
     <ros2_control name="GazeboSystem" type="system">
@@ -172,20 +242,20 @@
             <state_interface name="position"/>
             <state_interface name="velocity"/>
-         </joint>
+        </joint>
         <joint name="chassis_to_wheel_b">
                <command_interface name="velocity"/>
             <state_interface name="position"/>
             <state_interface name="velocity"/>
-         </joint>
+        </joint>
         <joint name="chassis_to_wheel_c">
                <command_interface name="velocity"/>
             <state_interface name="position"/>
             <state_interface name="velocity"/>
-         </joint>
+        </joint>
         <joint name="chassis_to_wheel_d">
                <command_interface name="velocity"/>
             <state_interface name="position"/>
             <state_interface name="velocity"/>
-         </joint>
+        </joint>
     </ros2_control>
     <!-- Gazebo Sim Plugins -->

Commit message: fixed collision model + rotated cameras correctly

File: robot/x_drive.urdf.xacro (robot description, xacro)
@@ -32,7 +32,7 @@
             </geometry>
             -->
-            <origin xyz="0 0 0.25" rpy="0 0 0"/>
-            <geometry>
-                <cylinder length="0.0315" radius="0.055"/>
+            <origin xyz="0 0 0.05" rpy="0 0 0"/>
+            <geometry>
+                 <box size='0.20 0.20 0.02'/>
             </geometry>
         </collision>
@@ -41,5 +41,5 @@
             <mass value="4.54"/>
            <inertia
-                  ixx="0.05487"
+                ixx="0.05487"
                 ixy="0.0"
                 ixz="0.0"
@@ -62,5 +62,5 @@
             </visual>
             <collision>
-                <origin xyz="0.015 0 -0.0065" rpy="0 0 0"/>
+                <origin xyz="0 0 0" rpy="0 0 0"/>
                 <geometry>
                     <cylinder length="0.0315" radius="0.055"/>
@@ -168,5 +168,5 @@
                 <pose>0 0 0 0 0 0</pose>
                 <camera>
-                    <horizontal_fov>1.047</horizontal_fov>
+                    <horizontal_fov>1.0</horizontal_fov>
                     <image>
                         <width>${px_w}</width>
@@ -180,5 +180,5 @@
                 </camera>
                 <always_on>true</always_on>
-                <update_rate>30</update_rate>
+                <update_rate>10</update_rate> <!-- i think our cameras run at 90fps max, but for sim 30 kills it. maybe 10 will be better? -->
                 <visualize>true</visualize>
                 <topic>/${camera_name}/image_raw</topic>
@@ -188,8 +188,8 @@
     </xacro:macro>
     <!-- make sure to update ROS bridge in spawn_robot.launch.py! -->
-    <xacro:usb_cam camera_name='cam1' px_w='1920' px_h='1200' xyz='0.1 0 0.1' rpy='0 0 0'/>
-    <xacro:usb_cam camera_name='cam2' px_w='1920' px_h='1200' xyz='-0.1 0 0.1' rpy='0 0 ${pi}'/>
-    <xacro:usb_cam camera_name='cam3' px_w='1920' px_h='1200' xyz='0 0.1 0.1' rpy='0 0 ${pi/2}'/>
-    <xacro:usb_cam camera_name='cam4' px_w='1920' px_h='1200' xyz='0 -0.1 0.1' rpy='0 0 -${pi/2}'/>
+    <xacro:usb_cam camera_name='cam1' px_w='1920' px_h='1200' xyz='-0.08 0.08 0.1' rpy='0 0 ${3*pi/4}'/>
+    <xacro:usb_cam camera_name='cam2' px_w='1920' px_h='1200' xyz='-0.08 -0.08 0.1' rpy='0 0 -${3*pi/4}'/>
+    <xacro:usb_cam camera_name='cam3' px_w='1920' px_h='1200' xyz='0.08 0.08 0.1' rpy='0 0 ${pi/4}'/>
+    <xacro:usb_cam camera_name='cam4' px_w='1920' px_h='1200' xyz='0.08 -0.08 0.1' rpy='0 0 -${pi/4}'/>
     <!-- Joints -->
     <joint name="footprint_2_link" type='fixed'>
@@ -239,20 +239,20 @@
         </hardware>
         <joint name="chassis_to_wheel_a">
-               <command_interface name="velocity"/>
+            <command_interface name="velocity"/>
             <state_interface name="position"/>
             <state_interface name="velocity"/>
         </joint>
         <joint name="chassis_to_wheel_b">
-               <command_interface name="velocity"/>
+            <command_interface name="velocity"/>
             <state_interface name="position"/>
             <state_interface name="velocity"/>
         </joint>
         <joint name="chassis_to_wheel_c">
-               <command_interface name="velocity"/>
+            <command_interface name="velocity"/>
             <state_interface name="position"/>
             <state_interface name="velocity"/>
         </joint>
         <joint name="chassis_to_wheel_d">
-               <command_interface name="velocity"/>
+            <command_interface name="velocity"/>
             <state_interface name="position"/>
             <state_interface name="velocity"/>

Commit message: updated camera positions to match CAD model

File: robot/x_drive.urdf.xacro (robot description, xacro)
@@ -5,7 +5,12 @@
     <xacro:property name="model_path" value="package://robot_description/models"/>
     <xacro:property name="package_path" value="package://robot_gazebo/config"/>
+    <!--Wheel properties-->
     <xacro:property name="wheel_offs" value="0.14"/>
     <xacro:property name="wheel_rad" value="0.0349253"/>
     <xacro:property name="wheel_width" value="0.02159"/>
+    <!-- Camera properties-->
+    <xacro:property name="camera_x" value="0.114"/>
+    <xacro:property name="camera_y" value="0.116"/>
+    <xacro:property name="camera_z" value="0.197"/>
     <!--world link-->
     <link name='base_footprint'/>
@@ -49,6 +54,7 @@
             </inertial>
     </link>
-    <!--Sensor links-->
+    <!--imu link-->
     <link name="imu_link"/>
+    <!-- LiDAR -->
     <link name="laser_frame">
             <visual>
@@ -123,5 +129,5 @@
     <xacro:wheel_link name="wheel_d"/>
     <!-- Camera Xacro -->
-    <xacro:macro name='usb_cam' params='camera_name xyz rpy px_w px_h'>
+    <xacro:macro name='usb_cam' params='camera_name xyz rpy'>
         <link name='${camera_name}_link'>
             <visual>
@@ -168,17 +174,17 @@
                 <pose>0 0 0 0 0 0</pose>
                 <camera>
-                    <horizontal_fov>1.0</horizontal_fov>
+                    <horizontal_fov>1.26</horizontal_fov>
                     <image>
-                        <width>${px_w}</width>
-                        <height>${px_h}</height>
+                        <width>1920</width>
+                        <height>1200</height>
                         <format>R8G8B8</format>
                     </image>
                     <clip>
-                        <near>0.1</near>
-                        <far>100</far>
+                        <near>0.001</near>
+                        <far>20</far>
                     </clip>
                 </camera>
                 <always_on>true</always_on>
-                <update_rate>10</update_rate> <!-- i think our cameras run at 90fps max, but for sim 30 kills it. maybe 10 will be better? -->
+                <update_rate>10</update_rate> <!-- i think our cameras run at 90fps max, but for sim, even 30 kills it. maybe 10 will be better? -->
                 <visualize>true</visualize>
                 <topic>/${camera_name}/image_raw</topic>
@@ -188,8 +194,8 @@
     </xacro:macro>
     <!-- make sure to update ROS bridge in spawn_robot.launch.py! -->
-    <xacro:usb_cam camera_name='cam1' px_w='1920' px_h='1200' xyz='-0.08 0.08 0.2' rpy='0 0 ${3*pi/4}'/>
-    <xacro:usb_cam camera_name='cam2' px_w='1920' px_h='1200' xyz='-0.08 -0.08 0.2' rpy='0 0 -${3*pi/4}'/>
-    <xacro:usb_cam camera_name='cam3' px_w='1920' px_h='1200' xyz='0.08 0.08 0.2' rpy='0 0 ${pi/4}'/>
-    <xacro:usb_cam camera_name='cam4' px_w='1920' px_h='1200' xyz='0.08 -0.08 0.2' rpy='0 0 -${pi/4}'/>
+    <xacro:usb_cam camera_name='cam1' xyz='-${camera_x} ${camera_y} ${camera_z}' rpy='0 0 ${3*pi/4}'/>
+    <xacro:usb_cam camera_name='cam2' xyz='-${camera_x} -${camera_y} ${camera_z}' rpy='0 0 -${3*pi/4}'/>
+    <xacro:usb_cam camera_name='cam3' xyz='${camera_x} ${camera_y} ${camera_z}' rpy='0 0 ${pi/4}'/>
+    <xacro:usb_cam camera_name='cam4' xyz='${camera_x} -${camera_y} ${camera_z}' rpy='0 0 -${pi/4}'/>
     <!-- Joints -->
     <joint name="footprint_2_link" type='fixed'>
@@ -231,5 +237,5 @@
         <parent link="base_link"/>
         <child link="laser_frame"/>
-        <origin xyz="0 0 0.2" rpy="0 0 0"/>
+        <origin xyz="0 0 0.1" rpy="0 0 0"/>
     </joint>
     <!-- ROS 2 Control-->
