Commit message: have 2 working lidars

File: robot/x_drive.urdf.xacro (robot description, xacro)
@@ -56,33 +56,4 @@
     <!--imu link-->
     <link name="imu_link"/>
-    <!-- LiDAR -->
-    <link name="laser_frame">
-            <visual>
-                <origin xyz="0 0 0.0" rpy="0 0 0"/>
-                <geometry>
-                    <cylinder length="0.0315" radius="0.055"/>
-                </geometry>
-                <material name="dark_grey">
-                    <color rgba="0.2 0.2 0.2 1.0"/>
-                </material>
-            </visual>
-            <collision>
-                <origin xyz="0 0 0" rpy="0 0 0"/>
-                <geometry>
-                    <cylinder length="0.0315" radius="0.055"/>
-                </geometry>
-            </collision>
-            <inertial>
-                <origin xyz="0 0 0" />
-                <mass value="0.114" />
-                <inertia
-                ixx="0.001"
-                ixy="0.0"
-                ixz="0.0"
-                iyy="0.001"
-                iyz="0.0"
-                izz="0.001"/>
-            </inertial>
-    </link>
     <!-- wheels -->
     <xacro:macro name="wheel_link" params="name">
@@ -128,5 +99,5 @@
     <xacro:wheel_link name="wheel_c"/>
     <xacro:wheel_link name="wheel_d"/>
-    <!-- Camera Xacro -->
+    <!-- USB Camera x4 -->
     <xacro:macro name='usb_cam' params='camera_name xyz rpy'>
         <link name='${camera_name}_link'>
@@ -198,4 +169,75 @@
     <xacro:usb_cam camera_name='cam3' xyz='${camera_x} ${camera_y} ${camera_z}' rpy='0 0 ${pi/4}'/>
     <xacro:usb_cam camera_name='cam4' xyz='${camera_x} -${camera_y} ${camera_z}' rpy='0 0 -${pi/4}'/>
+    <!-- LiDAR x2 -->
+    <xacro:macro name='TiMXXS_lidar' params='sensor_number xyz yaw'>
+        <!-- lidar link -->
+        <link name="laser_frame_${sensor_number}">
+            <visual>
+                <origin xyz="0 0 0.0" rpy="0 0 0"/>
+                <geometry>
+                    <cylinder length="0.02" radius="0.02"/>
+                </geometry>
+                <material name="dark_grey">
+                    <color rgba="0.2 0.2 0.2 1.0"/>
+                </material>
+            </visual>
+            <collision>
+                <origin xyz="0 0 0" rpy="0 0 0"/>
+                <geometry>
+                    <cylinder length="0.02" radius="0.02"/>
+                </geometry>
+            </collision>
+            <inertial>
+                <origin xyz="0 0 0" />
+                <mass value="0.114" />
+                <inertia
+                ixx="0.001"
+                ixy="0.0"
+                ixz="0.0"
+                iyy="0.001"
+                iyz="0.0"
+                izz="0.001"/>
+            </inertial>
+        </link>
+        <!-- lidar joint -->
+        <joint name="laser_joint_${sensor_number}" type="fixed">
+            <parent link="base_link"/>
+            <child link="laser_frame_${sensor_number}"/>
+            <origin xyz="${xyz}" rpy="0 0 ${yaw}"/>
+        </joint>
+        <!-- actual sensor-->
+        <gazebo reference="laser_frame_${sensor_number}">
+            <sensor name="lidar_${sensor_number}" type="gpu_lidar">
+                <pose>0 0 0 0 0 0</pose>
+                <always_on>true</always_on>
+                <visualize>true</visualize>
+                <update_rate>10</update_rate>
+                <topic>scan_${sensor_number}</topic>
+                <gz_frame_id>laser_frame_${sensor_number}</gz_frame_id>
+                <lidar>
+                    <scan>
+                        <horizontal>
+                            <samples>720</samples>
+                            <resolution>1</resolution>
+                            <min_angle>-0.785398163</min_angle>
+                            <max_angle>3.92699</max_angle>
+                        </horizontal>
+                    </scan>
+                    <range>
+                        <min>0.15</min>
+                        <max>10.0</max>
+                        <resolution>0.01</resolution>
+                    </range>
+                    <noise>
+                        <type>gaussian</type>
+                        <mean>0.0</mean>
+                        <stddev>0.01</stddev>
+                    </noise>
+                </lidar>
+            </sensor>
+        </gazebo>
+    </xacro:macro>
+    <xacro:TiMXXS_lidar sensor_number='1' xyz="0.13 0.12 0.14" yaw='-${pi/4}'/>
+    <xacro:TiMXXS_lidar sensor_number='2' xyz="-0.13 0.12 0.14" yaw='${pi/4}'/>
     <!-- Joints -->
     <joint name="footprint_2_link" type='fixed'>
@@ -233,9 +275,4 @@
         <child link="imu_link"/>
         <origin xyz="0 0 0.04" rpy="0 0 0"/>
-    </joint>
-    <joint name="laser_joint" type="fixed">
-        <parent link="base_link"/>
-        <child link="laser_frame"/>
-        <origin xyz="0 0 0.1" rpy="0 0 0"/>
     </joint>
     <!-- ROS 2 Control-->
@@ -271,41 +308,3 @@
           </plugin>
     </gazebo>
-    <!-- Sensor Gazebo Tag-->
-    <gazebo reference="laser_frame">
-        <sensor name="lidar" type="gpu_lidar">
-            <pose>0 0 0 0 0 0</pose>
-            <always_on>true</always_on>
-            <visualize>true</visualize>
-            <update_rate>10</update_rate>
-            <topic>scan</topic>
-            <gz_frame_id>laser_frame</gz_frame_id>
-            <lidar>
-                <scan>
-                    <horizontal>
-                        <samples>720</samples>
-                        <resolution>1</resolution>
-                        <min_angle>-3.14</min_angle>
-                        <max_angle>3.14</max_angle>
-                    </horizontal>
-                </scan>
-                <range>
-                    <min>0.05</min>
-                    <max>10.0</max>
-                    <resolution>0.01</resolution>
-                </range>
-                <noise>
-                    <type>gaussian</type>
-                    <mean>0.0</mean>
-                    <stddev>0.01</stddev>
-                </noise>
-            </lidar>
-        </sensor>
-    </gazebo>
-<!-- This might cause problems later...
-[gazebo-1] Warning [Utils.cc:132] [/sdf/model[@name="x_drive"]/link[@name="base_footprint"]/sensor[@name="cam1_sensor"]/gz_frame_id:<data-string>:L207]: XML Element[gz_frame_id], child of element[sensor], not defined in SDF. Copying[gz_frame_id] as children of [sensor].
-[gazebo-1] Warning [Utils.cc:132] [/sdf/model[@name="x_drive"]/link[@name="base_footprint"]/sensor[@name="cam2_sensor"]/gz_frame_id:<data-string>:L227]: XML Element[gz_frame_id], child of element[sensor], not defined in SDF. Copying[gz_frame_id] as children of [sensor].
-[gazebo-1] Warning [Utils.cc:132] [/sdf/model[@name="x_drive"]/link[@name="base_footprint"]/sensor[@name="cam3_sensor"]/gz_frame_id:<data-string>:L247]: XML Element[gz_frame_id], child of element[sensor], not defined in SDF. Copying[gz_frame_id] as children of [sensor].
-[gazebo-1] Warning [Utils.cc:132] [/sdf/model[@name="x_drive"]/link[@name="base_footprint"]/sensor[@name="cam4_sensor"]/gz_frame_id:<data-string>:L267]: XML Element[gz_frame_id], child of element[sensor], not defined in SDF. Copying[gz_frame_id] as children of [sensor].
-[gazebo-1] Warning [Utils.cc:132] [/sdf/model[@name="x_drive"]/link[@name="base_footprint"]/sensor[@name="lidar"]/gz_frame_id:<data-string>:L295]: XML Element[gz_frame_id], child of element[sensor], not defined in SDF. Copying[gz_frame_id] as children of [sensor].
--->
 </robot>

Commit message: fixed lidar rotation + position

File: robot/x_drive.urdf.xacro (robot description, xacro)
@@ -18,9 +18,4 @@
     <link name="base_link">
         <visual>
-            <!--
-            <geometry>
-                <mesh filename='${model_path}/chassis-v2.dae'/>
-            </geometry>
-            -->
             <origin xyz="0 0 0.05" rpy="0 0 0"/>
             <geometry>
@@ -32,9 +27,4 @@
         </visual>
         <collision>
-            <!--
-            <geometry>
-                <mesh filename='${model_path}/chassis.dae'/>
-            </geometry>
-            -->
             <origin xyz="0 0 0.05" rpy="0 0 0"/>
             <geometry>
@@ -238,6 +228,6 @@
         </gazebo>
     </xacro:macro>
-    <xacro:TiMXXS_lidar sensor_number='1' xyz="0.13 0.12 0.14" yaw='-${pi/4}'/>
-    <xacro:TiMXXS_lidar sensor_number='2' xyz="-0.13 0.12 0.14" yaw='${pi/4}'/>
+    <xacro:TiMXXS_lidar sensor_number='1' xyz="-0.13 0.12 0.14" yaw='${3* pi/4}'/>
+    <xacro:TiMXXS_lidar sensor_number='2' xyz="-0.13 -0.12 0.14" yaw='-${ 3* pi/4}'/>
     <!-- Joints -->
     <joint name="footprint_2_link" type='fixed'>

Commit message: box representing intake has been added

File: robot/x_drive.urdf.xacro (robot description, xacro)
@@ -44,4 +44,32 @@
             </inertial>
     </link>
+    <link name="intake_link">
+        <visual>
+            <origin xyz='0 0 0' rpy='0 0 0'/>
+            <geometry>
+                <box size='0.189 0.146 0.20'/>
+            </geometry>
+            <material name="light-blue">
+                <color rgba="0.68 0.85 0.9 1"/>
+            </material>
+        </visual>
+        <collision>
+            <origin xyz="0 0 0" rpy="0 0 0"/>
+            <geometry>
+                <box size='0.189 0.146 0.10'/>
+            </geometry>
+        </collision>
+        <inertial>
+            <origin xyz="0 0 0" rpy="0 0 0"/>
+            <mass value="0.070"/>
+            <inertia
+            ixx="0.001"
+            ixy="0.0"
+            ixz="0.0"
+            iyy="0.001"
+            iyz="0.0"
+            izz="0.001"/>
+        </inertial>
+    </link>
     <!--imu link-->
     <link name="imu_link"/>
@@ -236,4 +264,9 @@
         <child link='base_link'/>
     </joint>
+    <joint name="base_2_intake" type='fixed'>
+        <origin xyz="0.0945 0 0.16" rpy="0 0 0"/>
+        <parent link='base_link'/>
+        <child link='intake_link'/>
+    </joint>
     <joint name="chassis_to_wheel_a" type="continuous">
         <origin xyz="-${wheel_offs} ${wheel_offs} ${wheel_rad}" rpy="0 0 ${pi/4}"/>
