Commit message: node initializes, robot jumpy
sucessfully got robot_localization package to load and not crash. robot is super jumpy when turning, pretty good when driving in a line.

File: robot/otto_lite.urdf.xacro (robot description, xacro)
@@ -44,5 +44,5 @@
             <origin xyz='0 0 0' rpy='0 0 0'/>
             <geometry>
-                <box size='0.189 0.146 0.20'/>
+                <box size='0.189 0.146 0.10'/>
             </geometry>
             <material name="light-blue">
@@ -68,4 +68,6 @@
         </inertial>
     </link>
+    <!--for scoring.py purposes-->
+    <link name="intake_reference"/>
     <!--imu link-->
     <link name="imu_link"/>
@@ -245,4 +247,11 @@
         <child link='intake_link'/>
     </joint>
+    <!--for scoring.py purposes-->
+    <joint name="base_2_ref" type="fixed">
+        <origin xyz="0.189 0 0" rpy="0 0 0"/>
+        <parent link="base_link"/>
+        <child link="intake_reference"/>
+    </joint>
+    <!--Continuous Joints-->
     <joint name="chassis_to_wheel_a" type="continuous">
         <origin xyz="-${wheel_offs} ${wheel_offs} ${wheel_rad}" rpy="0 0 ${pi/4}"/>
