Commit message: changed wheel joint names in urdf

File: robot/logical_cameras.urdf.xacro (robot description, xacro)
@@ -1,10 +1,10 @@
 <?xml version='1.0'?>
 <robot xmlns:xacro="http://www.ros.org/wiki/xacro" xmlns:gz="http://gazebosim.org/schema">
-   <!-- Camera properties-->
+    <!-- Camera properties-->
     <xacro:property name="camera_x" value="0.114"/>
     <xacro:property name="camera_y" value="0.116"/>
     <xacro:property name="camera_z" value="0.197"/>
     <xacro:property name='tilt_angle' value=' 0.122'/> <!--this is the p value in rpy!-->
-<!-- USB Camera x4 -->
+    <!-- USB Camera x4 -->
     <xacro:macro name='logical_cam' params='camera_name xyz rpy'>
         <link name='${camera_name}_link'>
@@ -62,5 +62,5 @@
         </gazebo>
     </xacro:macro>
-        <!-- make sure to update ROS bridge in spawn_robot.launch.py! -->
+    <!-- make sure to update ROS bridge in spawn_robot.launch.py! -->
     <xacro:logical_cam camera_name='cam1' xyz='-${camera_x} ${camera_y} ${camera_z}' rpy='0 ${tilt_angle} ${3*pi/4}'/>
     <xacro:logical_cam camera_name='cam2' xyz='-${camera_x} -${camera_y} ${camera_z}' rpy='0 ${tilt_angle} -${3*pi/4}'/>

File: robot/otto_lite.urdf.xacro (robot description, xacro)
@@ -162,7 +162,7 @@
     </xacro:macro>
     <xacro:wheel_link name="wheel_a"/>
-    <xacro:wheel_link name="wheel_b"/>
-    <xacro:wheel_link name="wheel_c"/>
-    <xacro:wheel_link name="wheel_d"/>
+    <xacro:wheel_link name="front_right_wheel"/>
+    <xacro:wheel_link name="front_left_wheel"/>
+    <xacro:wheel_link name="back_right_wheel"/>
     <!-- LiDAR x2 -->
     <xacro:macro name='TiMXXS_lidar' params='sensor_number xyz yaw'>
@@ -247,26 +247,26 @@
         <child link='intake_link'/>
     </joint>
-    <joint name="chassis_to_wheel_a" type="continuous">
+    <joint name="back_left_wheel_joint" type="continuous">
         <origin xyz="-${wheel_offs} ${wheel_offs} ${wheel_rad}" rpy="0 0 ${pi/4}"/>
         <parent link="base_link"/>
-        <child link="wheel_a"/>
+        <child link="back_left_wheel"/>
         <axis xyz="0 1 0"/>
     </joint>
-    <joint name="chassis_to_wheel_b" type="continuous">
+    <joint name="front_right_wheel_joint" type="continuous">
         <origin xyz="${wheel_offs} -${wheel_offs} ${wheel_rad}" rpy="0 0 ${-3* (pi/4)}"/>
         <parent link="base_link"/>
-        <child link="wheel_b"/>
+        <child link="front_right_wheel"/>
         <axis xyz="0 1 0"/>
     </joint>
-    <joint name="chassis_to_wheel_c" type="continuous">
+    <joint name="front_left_wheel_joint" type="continuous">
         <origin xyz="${wheel_offs} ${wheel_offs} ${wheel_rad}" rpy="0 0 -${pi/4}"/>
         <parent link="base_link"/>
-        <child link="wheel_c"/>
+        <child link="front_left_wheel"/>
         <axis xyz="0 1 0"/>
     </joint>
-    <joint name="chassis_to_wheel_d" type="continuous">
+    <joint name="back_right_wheel_joint" type="continuous">
         <origin xyz="-${wheel_offs} -${wheel_offs} ${wheel_rad}" rpy="0 0 ${3 *(pi/4)}"/>
         <parent link="base_link"/>
-        <child link="wheel_d"/>
+        <child link="back_right_wheel"/>
         <axis xyz="0 1 0"/>
     </joint>
@@ -282,20 +282,20 @@
             <plugin>gz_ros2_control/GazeboSimSystem</plugin>
         </hardware>
-        <joint name="chassis_to_wheel_a">
+        <joint name="back_left_wheel_joint">
             <command_interface name="velocity"/>
             <state_interface name="position"/>
             <state_interface name="velocity"/>
         </joint>
-        <joint name="chassis_to_wheel_b">
+        <joint name="front_right_wheel_joint">
             <command_interface name="velocity"/>
             <state_interface name="position"/>
             <state_interface name="velocity"/>
         </joint>
-        <joint name="chassis_to_wheel_c">
+        <joint name="front_left_wheel_joint">
             <command_interface name="velocity"/>
             <state_interface name="position"/>
             <state_interface name="velocity"/>
         </joint>
-        <joint name="chassis_to_wheel_d">
+        <joint name="back_right_wheel_joint">
             <command_interface name="velocity"/>
             <state_interface name="position"/>
