Commit message: made name changes, package builds

File: robot/otto.urdf.xacro (robot description, xacro)
@@ -1,12 +1,16 @@
 <?xml version='1.0'?>
-<robot name="x_drive_lite" xmlns:xacro="http://www.ros.org/wiki/xacro" xmlns:gz="http://gazebosim.org/schema">
+<robot name="Otto" xmlns:xacro="http://www.ros.org/wiki/xacro" xmlns:gz="http://gazebosim.org/schema">
     <static>false</static>
     <!-- properties-->
     <xacro:property name="model_path" value="package://robot_description/models"/>
-    <xacro:property name="package_path" value="package://robot_gazebo/config"/>
+    <xacro:property name="package_path" value="package://otto_gazebo/config"/>
     <!--Wheel properties-->
     <xacro:property name="wheel_offs" value="0.14"/>
     <xacro:property name="wheel_rad" value="0.0349253"/>
     <xacro:property name="wheel_width" value="0.02159"/>
+    <!-- Camera properties-->
+    <xacro:property name="camera_x" value="0.114"/>
+    <xacro:property name="camera_y" value="0.116"/>
+    <xacro:property name="camera_z" value="0.197"/>
     <!--world link-->
     <link name='base_footprint'/>
@@ -122,4 +126,74 @@
     <xacro:wheel_link name="wheel_c"/>
     <xacro:wheel_link name="wheel_d"/>
+    <!-- USB Camera x4 -->
+    <xacro:macro name='usb_cam' params='camera_name xyz rpy'>
+        <link name='${camera_name}_link'>
+            <visual>
+                <geometry>
+                    <box size='0.02 0.02 0.02'/>
+                </geometry>
+                <material name="dark_grey">
+                    <color rgba="0.2 0.2 0.2 1.0"/>
+                </material>
+            </visual>
+            <collision>
+                <geometry>
+                    <box size='0.02 0.02 0.02'/>
+                </geometry>
+                <material name="dark_grey">
+                    <color rgba="0.2 0.2 0.2 1.0"/>
+                </material>
+            </collision>
+            <inertial>
+                <origin xyz="0 0 0" rpy="0 0 0"/>
+                <mass value="0.01"/>
+                <inertia
+                    ixx="0.000001"
+                    ixy="0.0"
+                    ixz="0.0"
+                    iyy="0.000001"
+                    iyz="0.0"
+                    izz="0.000001"/>
+            </inertial>
+        </link>
+        <joint name="${camera_name}_joint" type="fixed">
+            <parent link="base_link"/>
+            <child link="${camera_name}_link"/>
+            <origin xyz="${xyz}" rpy="${rpy}"/>
+        </joint>
+        <link name="${camera_name}_link_optical"/>
+        <joint name="${camera_name}_optical_joint" type="fixed">
+            <parent link="${camera_name}_link"/>
+            <child link="${camera_name}_link_optical"/>
+            <origin xyz="0 0 0" rpy="-1.5708 0 -1.5708"/>
+        </joint>
+        <gazebo reference='${camera_name}_link'>
+            <sensor name='${camera_name}_sensor' type="camera">
+                <pose>0 0 0 0 0 0</pose>
+                <camera>
+                    <horizontal_fov>1.26</horizontal_fov>
+                    <image>
+                        <width>1920</width>
+                        <height>1200</height>
+                        <format>R8G8B8</format>
+                    </image>
+                    <clip>
+                        <near>0.001</near>
+                        <far>20</far>
+                    </clip>
+                </camera>
+                <always_on>true</always_on>
+                <update_rate>10</update_rate> <!-- i think our cameras run at 90fps max, but for sim, even 30 kills it. maybe 10 will be better? -->
+                <visualize>true</visualize>
+                <topic>/${camera_name}/image_raw</topic>
+                <gz_frame_id>${camera_name}_link_optical</gz_frame_id>
+            </sensor>
+        </gazebo>
+    </xacro:macro>
+    <!-- make sure to update ROS bridge in spawn_robot.launch.py! -->
+    <xacro:usb_cam camera_name='cam1' xyz='-${camera_x} ${camera_y} ${camera_z}' rpy='0 0 ${3*pi/4}'/>
+    <xacro:usb_cam camera_name='cam2' xyz='-${camera_x} -${camera_y} ${camera_z}' rpy='0 0 -${3*pi/4}'/>
+    <xacro:usb_cam camera_name='cam3' xyz='${camera_x} ${camera_y} ${camera_z}' rpy='0 0 ${pi/4}'/>
+    <xacro:usb_cam camera_name='cam4' xyz='${camera_x} -${camera_y} ${camera_z}' rpy='0 0 -${pi/4}'/>
     <!-- LiDAR x2 -->
     <xacro:macro name='TiMXXS_lidar' params='sensor_number xyz yaw'>
@@ -263,5 +337,5 @@
     <gazebo>
           <plugin filename="gz_ros2_control-system" name="gz_ros2_control::GazeboSimROS2ControlPlugin">
-            <parameters>$(find robot_gazebo)/config/omni_wheel_params.yaml</parameters>
+            <parameters>$(find otto_gazebo)/config/omni_wheel_params.yaml</parameters>
           </plugin>
     </gazebo>

File: robot/otto_lite.urdf.xacro (robot description, xacro)
@@ -1,16 +1,12 @@
 <?xml version='1.0'?>
-<robot name="x_drive" xmlns:xacro="http://www.ros.org/wiki/xacro" xmlns:gz="http://gazebosim.org/schema">
+<robot name="Otto_lite" xmlns:xacro="http://www.ros.org/wiki/xacro" xmlns:gz="http://gazebosim.org/schema">
     <static>false</static>
     <!-- properties-->
     <xacro:property name="model_path" value="package://robot_description/models"/>
-    <xacro:property name="package_path" value="package://robot_gazebo/config"/>
+    <xacro:property name="package_path" value="package://otto_gazebo/config"/>
     <!--Wheel properties-->
     <xacro:property name="wheel_offs" value="0.14"/>
     <xacro:property name="wheel_rad" value="0.0349253"/>
     <xacro:property name="wheel_width" value="0.02159"/>
-    <!-- Camera properties-->
-    <xacro:property name="camera_x" value="0.114"/>
-    <xacro:property name="camera_y" value="0.116"/>
-    <xacro:property name="camera_z" value="0.197"/>
     <!--world link-->
     <link name='base_footprint'/>
@@ -126,74 +122,4 @@
     <xacro:wheel_link name="wheel_c"/>
     <xacro:wheel_link name="wheel_d"/>
-    <!-- USB Camera x4 -->
-    <xacro:macro name='usb_cam' params='camera_name xyz rpy'>
-        <link name='${camera_name}_link'>
-            <visual>
-                <geometry>
-                    <box size='0.02 0.02 0.02'/>
-                </geometry>
-                <material name="dark_grey">
-                    <color rgba="0.2 0.2 0.2 1.0"/>
-                </material>
-            </visual>
-            <collision>
-                <geometry>
-                    <box size='0.02 0.02 0.02'/>
-                </geometry>
-                <material name="dark_grey">
-                    <color rgba="0.2 0.2 0.2 1.0"/>
-                </material>
-            </collision>
-            <inertial>
-                <origin xyz="0 0 0" rpy="0 0 0"/>
-                <mass value="0.01"/>
-                <inertia
-                    ixx="0.000001"
-                    ixy="0.0"
-                    ixz="0.0"
-                    iyy="0.000001"
-                    iyz="0.0"
-                    izz="0.000001"/>
-            </inertial>
-        </link>
-        <joint name="${camera_name}_joint" type="fixed">
-            <parent link="base_link"/>
-            <child link="${camera_name}_link"/>
-            <origin xyz="${xyz}" rpy="${rpy}"/>
-        </joint>
-        <link name="${camera_name}_link_optical"/>
-        <joint name="${camera_name}_optical_joint" type="fixed">
-            <parent link="${camera_name}_link"/>
-            <child link="${camera_name}_link_optical"/>
-            <origin xyz="0 0 0" rpy="-1.5708 0 -1.5708"/>
-        </joint>
-        <gazebo reference='${camera_name}_link'>
-            <sensor name='${camera_name}_sensor' type="camera">
-                <pose>0 0 0 0 0 0</pose>
-                <camera>
-                    <horizontal_fov>1.26</horizontal_fov>
-                    <image>
-                        <width>1920</width>
-                        <height>1200</height>
-                        <format>R8G8B8</format>
-                    </image>
-                    <clip>
-                        <near>0.001</near>
-                        <far>20</far>
-                    </clip>
-                </camera>
-                <always_on>true</always_on>
-                <update_rate>10</update_rate> <!-- i think our cameras run at 90fps max, but for sim, even 30 kills it. maybe 10 will be better? -->
-                <visualize>true</visualize>
-                <topic>/${camera_name}/image_raw</topic>
-                <gz_frame_id>${camera_name}_link_optical</gz_frame_id>
-            </sensor>
-        </gazebo>
-    </xacro:macro>
-    <!-- make sure to update ROS bridge in spawn_robot.launch.py! -->
-    <xacro:usb_cam camera_name='cam1' xyz='-${camera_x} ${camera_y} ${camera_z}' rpy='0 0 ${3*pi/4}'/>
-    <xacro:usb_cam camera_name='cam2' xyz='-${camera_x} -${camera_y} ${camera_z}' rpy='0 0 -${3*pi/4}'/>
-    <xacro:usb_cam camera_name='cam3' xyz='${camera_x} ${camera_y} ${camera_z}' rpy='0 0 ${pi/4}'/>
-    <xacro:usb_cam camera_name='cam4' xyz='${camera_x} -${camera_y} ${camera_z}' rpy='0 0 -${pi/4}'/>
     <!-- LiDAR x2 -->
     <xacro:macro name='TiMXXS_lidar' params='sensor_number xyz yaw'>
@@ -337,5 +263,5 @@
     <gazebo>
           <plugin filename="gz_ros2_control-system" name="gz_ros2_control::GazeboSimROS2ControlPlugin">
-            <parameters>$(find robot_gazebo)/config/omni_wheel_params.yaml</parameters>
+            <parameters>$(find otto_gazebo)/config/omni_wheel_params.yaml</parameters>
           </plugin>
     </gazebo>

Commit message: refactored localization launch
added launch arguments for all config files and sim time

File: robot/otto.urdf.xacro (robot description, xacro)
@@ -3,5 +3,5 @@
     <static>false</static>
     <!-- properties-->
-    <xacro:property name="model_path" value="package://robot_description/models"/>
+    <xacro:property name="model_path" value="package://otto_description/models"/>
     <xacro:property name="package_path" value="package://otto_gazebo/config"/>
     <!--Wheel properties-->

File: robot/otto_lite.urdf.xacro (robot description, xacro)
@@ -3,5 +3,5 @@
     <static>false</static>
     <!-- properties-->
-    <xacro:property name="model_path" value="package://robot_description/models"/>
+    <xacro:property name="model_path" value="package://otto_description/models"/>
     <xacro:property name="package_path" value="package://otto_gazebo/config"/>
     <!--Wheel properties-->

Commit message: added 7 deg camera tilt

File: robot/otto.urdf.xacro (robot description, xacro)
@@ -13,4 +13,5 @@
     <xacro:property name="camera_y" value="0.116"/>
     <xacro:property name="camera_z" value="0.197"/>
+    <xacro:property name='tilt_angle' value=' 0.122'/> <!--this is the p value in rpy!-->
     <!--world link-->
     <link name='base_footprint'/>
@@ -141,7 +142,4 @@
                     <box size='0.02 0.02 0.02'/>
                 </geometry>
-                <material name="dark_grey">
-                    <color rgba="0.2 0.2 0.2 1.0"/>
-                </material>
             </collision>
             <inertial>
@@ -192,8 +190,8 @@
     </xacro:macro>
     <!-- make sure to update ROS bridge in spawn_robot.launch.py! -->
-    <xacro:usb_cam camera_name='cam1' xyz='-${camera_x} ${camera_y} ${camera_z}' rpy='0 0 ${3*pi/4}'/>
-    <xacro:usb_cam camera_name='cam2' xyz='-${camera_x} -${camera_y} ${camera_z}' rpy='0 0 -${3*pi/4}'/>
-    <xacro:usb_cam camera_name='cam3' xyz='${camera_x} ${camera_y} ${camera_z}' rpy='0 0 ${pi/4}'/>
-    <xacro:usb_cam camera_name='cam4' xyz='${camera_x} -${camera_y} ${camera_z}' rpy='0 0 -${pi/4}'/>
+    <xacro:usb_cam camera_name='cam1' xyz='-${camera_x} ${camera_y} ${camera_z}' rpy='0 ${tilt_angle} ${3*pi/4}'/>
+    <xacro:usb_cam camera_name='cam2' xyz='-${camera_x} -${camera_y} ${camera_z}' rpy='0 ${tilt_angle} -${3*pi/4}'/>
+    <xacro:usb_cam camera_name='cam3' xyz='${camera_x} ${camera_y} ${camera_z}' rpy='0 ${tilt_angle} ${pi/4}'/>
+    <xacro:usb_cam camera_name='cam4' xyz='${camera_x} -${camera_y} ${camera_z}' rpy='0 ${tilt_angle} -${pi/4}'/>
     <!-- LiDAR x2 -->
     <xacro:macro name='TiMXXS_lidar' params='sensor_number xyz yaw'>

Commit message: mppi drives faster

File: robot/otto.urdf.xacro (robot description, xacro)
@@ -379,3 +379,11 @@
           </plugin>
     </gazebo>
+    <gazebo>
+        <plugin
+            filename="gz-sim-pose-publisher-system"
+            name="gz::sim::systems::PosePublisher">
+            <use_pose_vector_msg>true</use_pose_vector_msg>
+            <publish_model_pose>true</publish_model_pose>
+        </plugin>
+    </gazebo>
 </robot>

File: robot/otto_lite.urdf.xacro (robot description, xacro)
@@ -72,5 +72,5 @@
     <!-- IMU -->
     <gazebo reference='imu_link'>
-         <sensor name="tb3_imu" type="imu"> <!--taken from turtlebot3_simulations-->
+        <sensor name="tb3_imu" type="imu"> <!--taken from turtlebot3_simulations-->
         <always_on>true</always_on>
         <update_rate>200</update_rate>
@@ -271,7 +271,7 @@
     <!--Sensor Joints-->
     <joint name="imu_joint" type="fixed">
+        <origin xyz="0 0 0.04" rpy="0 0 0"/>
         <parent link="base_link"/>
         <child link="imu_link"/>
-        <origin xyz="0 0 0.04" rpy="0 0 0"/>
     </joint>
     <!-- ROS 2 Control-->
@@ -307,3 +307,11 @@
           </plugin>
     </gazebo>
+    <gazebo>
+        <plugin
+            filename="gz-sim-pose-publisher-system"
+            name="gz::sim::systems::PosePublisher">
+            <use_pose_vector_msg>true</use_pose_vector_msg>
+            <publish_model_pose>true</publish_model_pose>
+        </plugin>
+    </gazebo>
 </robot>

Commit message: fixed nav2 config

File: robot/otto.urdf.xacro (robot description, xacro)
@@ -9,9 +9,6 @@
     <xacro:property name="wheel_rad" value="0.0349253"/>
     <xacro:property name="wheel_width" value="0.02159"/>
-    <!-- Camera properties-->
-    <xacro:property name="camera_x" value="0.114"/>
-    <xacro:property name="camera_y" value="0.116"/>
-    <xacro:property name="camera_z" value="0.197"/>
-    <xacro:property name='tilt_angle' value=' 0.122'/> <!--this is the p value in rpy!-->
+     <!--Robot Camera Properties -->
+    <xacro:include filename="$(find otto_gazebo)/robot/robot_cams.urdf.xacro"/>
     <!--world link-->
     <link name='base_footprint'/>
@@ -164,75 +161,8 @@
         </gazebo>
     </xacro:macro>
-    <xacro:wheel_link name="wheel_a"/>
-    <xacro:wheel_link name="wheel_b"/>
-    <xacro:wheel_link name="wheel_c"/>
-    <xacro:wheel_link name="wheel_d"/>
-    <!-- USB Camera x4 -->
-    <xacro:macro name='usb_cam' params='camera_name xyz rpy'>
-        <link name='${camera_name}_link'>
-            <visual>
-                <geometry>
-                    <box size='0.02 0.02 0.02'/>
-                </geometry>
-                <material name="dark_grey">
-                    <color rgba="0.2 0.2 0.2 1.0"/>
-                </material>
-            </visual>
-            <collision>
-                <geometry>
-                    <box size='0.02 0.02 0.02'/>
-                </geometry>
-            </collision>
-            <inertial>
-                <origin xyz="0 0 0" rpy="0 0 0"/>
-                <mass value="0.01"/>
-                <inertia
-                    ixx="0.000001"
-                    ixy="0.0"
-                    ixz="0.0"
-                    iyy="0.000001"
-                    iyz="0.0"
-                    izz="0.000001"/>
-            </inertial>
-        </link>
-        <joint name="${camera_name}_joint" type="fixed">
-            <parent link="base_link"/>
-            <child link="${camera_name}_link"/>
-            <origin xyz="${xyz}" rpy="${rpy}"/>
-        </joint>
-        <link name="${camera_name}_link_optical"/>
-        <joint name="${camera_name}_optical_joint" type="fixed">
-            <parent link="${camera_name}_link"/>
-            <child link="${camera_name}_link_optical"/>
-            <origin xyz="0 0 0" rpy="-1.5708 0 -1.5708"/>
-        </joint>
-        <gazebo reference='${camera_name}_link'>
-            <sensor name='${camera_name}_sensor' type="camera">
-                <pose>0 0 0 0 0 0</pose>
-                <camera>
-                    <horizontal_fov>1.26</horizontal_fov>
-                    <image>
-                        <width>1920</width>
-                        <height>1200</height>
-                        <format>R8G8B8</format>
-                    </image>
-                    <clip>
-                        <near>0.001</near>
-                        <far>20</far>
-                    </clip>
-                </camera>
-                <always_on>true</always_on>
-                <update_rate>10</update_rate> <!-- i think our cameras run at 90fps max, but for sim, even 30 kills it. maybe 10 will be better? -->
-                <visualize>true</visualize>
-                <topic>/${camera_name}/image_raw</topic>
-                <gz_frame_id>${camera_name}_link_optical</gz_frame_id>
-            </sensor>
-        </gazebo>
-    </xacro:macro>
-    <!-- make sure to update ROS bridge in spawn_robot.launch.py! -->
-    <xacro:usb_cam camera_name='cam1' xyz='-${camera_x} ${camera_y} ${camera_z}' rpy='0 ${tilt_angle} ${3*pi/4}'/>
-    <xacro:usb_cam camera_name='cam2' xyz='-${camera_x} -${camera_y} ${camera_z}' rpy='0 ${tilt_angle} -${3*pi/4}'/>
-    <xacro:usb_cam camera_name='cam3' xyz='${camera_x} ${camera_y} ${camera_z}' rpy='0 ${tilt_angle} ${pi/4}'/>
-    <xacro:usb_cam camera_name='cam4' xyz='${camera_x} -${camera_y} ${camera_z}' rpy='0 ${tilt_angle} -${pi/4}'/>
+    <xacro:wheel_link name="back_left_wheel"/>
+    <xacro:wheel_link name="front_right_wheel"/>
+    <xacro:wheel_link name="front_left_wheel"/>
+    <xacro:wheel_link name="back_right_wheel"/>
     <!-- LiDAR x2 -->
     <xacro:macro name='TiMXXS_lidar' params='sensor_number xyz yaw'>
@@ -317,26 +247,26 @@
         <child link='intake_link'/>
     </joint>
-    <joint name="chassis_to_wheel_a" type="continuous">
+    <joint name="back_left_wheel_joint" type="continuous">
         <origin xyz="-${wheel_offs} ${wheel_offs} ${wheel_rad}" rpy="0 0 ${pi/4}"/>
         <parent link="base_link"/>
-        <child link="wheel_a"/>
+        <child link="back_left_wheel"/>
         <axis xyz="0 1 0"/>
     </joint>
-    <joint name="chassis_to_wheel_b" type="continuous">
+    <joint name="front_right_wheel_joint" type="continuous">
         <origin xyz="${wheel_offs} -${wheel_offs} ${wheel_rad}" rpy="0 0 ${-3* (pi/4)}"/>
         <parent link="base_link"/>
-        <child link="wheel_b"/>
+        <child link="front_right_wheel"/>
         <axis xyz="0 1 0"/>
     </joint>
-    <joint name="chassis_to_wheel_c" type="continuous">
+    <joint name="front_left_wheel_joint" type="continuous">
         <origin xyz="${wheel_offs} ${wheel_offs} ${wheel_rad}" rpy="0 0 -${pi/4}"/>
         <parent link="base_link"/>
-        <child link="wheel_c"/>
+        <child link="front_left_wheel"/>
         <axis xyz="0 1 0"/>
     </joint>
-    <joint name="chassis_to_wheel_d" type="continuous">
+    <joint name="back_right_wheel_joint" type="continuous">
         <origin xyz="-${wheel_offs} -${wheel_offs} ${wheel_rad}" rpy="0 0 ${3 *(pi/4)}"/>
         <parent link="base_link"/>
-        <child link="wheel_d"/>
+        <child link="back_right_wheel"/>
         <axis xyz="0 1 0"/>
     </joint>
@@ -352,20 +282,20 @@
             <plugin>gz_ros2_control/GazeboSimSystem</plugin>
         </hardware>
-        <joint name="chassis_to_wheel_a">
+        <joint name="back_left_wheel_joint">
             <command_interface name="velocity"/>
             <state_interface name="position"/>
             <state_interface name="velocity"/>
         </joint>
-        <joint name="chassis_to_wheel_b">
+        <joint name="front_right_wheel_joint">
             <command_interface name="velocity"/>
             <state_interface name="position"/>
             <state_interface name="velocity"/>
         </joint>
-        <joint name="chassis_to_wheel_c">
+        <joint name="front_left_wheel_joint">
             <command_interface name="velocity"/>
             <state_interface name="position"/>
             <state_interface name="velocity"/>
         </joint>
-        <joint name="chassis_to_wheel_d">
+        <joint name="back_right_wheel_joint">
             <command_interface name="velocity"/>
             <state_interface name="position"/>
@@ -376,5 +306,5 @@
     <gazebo>
           <plugin filename="gz_ros2_control-system" name="gz_ros2_control::GazeboSimROS2ControlPlugin">
-            <parameters>$(find otto_gazebo)/config/omni_wheel_params.yaml</parameters>
+            <parameters>$(find otto_gazebo)/config/ros2_control.yaml</parameters>
           </plugin>
     </gazebo>

File: robot/otto_lite.urdf.xacro (robot description, xacro)
@@ -9,6 +9,5 @@
     <xacro:property name="wheel_rad" value="0.0349253"/>
     <xacro:property name="wheel_width" value="0.02159"/>
-    <!--logical camera include file-->
-    <!-- <xacro:include filename="$(find otto_gazebo)/robot/logical_cameras.urdf.xacro"/> -->
+    <!-- <xacro:include filename="$(find otto_gazebo)/robot/robot_cams.urdf.xacro"/> -->
     <!--world link-->
     <link name='base_footprint'/>
@@ -306,5 +305,5 @@
     <gazebo>
           <plugin filename="gz_ros2_control-system" name="gz_ros2_control::GazeboSimROS2ControlPlugin">
-            <parameters>$(find otto_gazebo)/config/omni_wheel_params.yaml</parameters>
+            <parameters>$(find otto_gazebo)/config/ros2_control.yaml</parameters>
           </plugin>
     </gazebo>
